Commit message: Made code more beautiful

File: spot/src/myrobot/urdf/thespot.urdf.xacro (robot description, xacro)
@@ -6,36 +6,36 @@
   			 	<child link="body"/>
   			</joint>
-		<link name ="body">
-			<visual>
-      	<origin xyz="0 0 0.3" rpy="0 0 0" />
-       		<geometry>
-          	<box size="0.4 0.2 0.1" />
-        	</geometry>
-        	<material name="Cyan">
-          	<color rgba="0 1.0 1.0 1.0"/>
-       		</material>
-      </visual>
-			<inertial>
-				<mass value="5"/>
-				<inertia ixx="0.1" ixy="0.0" ixz="0.1" iyy="0.0" iyz="0.0" izz="0.1"/>
-			</inertial>
-			<collision>
-	<origin xyz="0 0 0.3" rpy="0 0 0" />
-       				<geometry>
-          	<box size="0.4 0.2 0.1" />
-        	</geometry>
-			</collision>
-		</link>
-			<xacro:macro name="leg" params="prefix reflect_big_link reflect_big_joint reflect_small_link  reflect_small_joint">
-		<link name="${prefix}_big_leg">
-			<visual>
-				<origin xyz="${reflect_big_link}" rpy="0 -0.7 0" />
-       		<geometry>
-          	<box size="0.2 0.03 0.03" />
-        	</geometry>
+			<link name ="body">
+				<visual>
+      					<origin xyz="0 0 0.3" rpy="0 0 0" />
+       					<geometry>
+          					<box size="0.4 0.2 0.1" />
+        				</geometry>
+        				<material name="Cyan">
+          					<color rgba="0 1.0 1.0 1.0"/>
+       					</material>
+      				</visual>
+				<inertial>
+					<mass value="5"/>
+					<inertia ixx="0.1" ixy="0.0" ixz="0.1" iyy="0.0" iyz="0.0" izz="0.1"/>
+				</inertial>
+				<collision>
+					<origin xyz="0 0 0.3" rpy="0 0 0" />
+       					<geometry>
+          					<box size="0.4 0.2 0.1" />
+        				</geometry>
+				</collision>
+			</link>
+<xacro:macro name="leg" params="prefix reflect_big_link reflect_big_joint reflect_small_link  reflect_small_joint">
+	<link name="${prefix}_big_leg">
+		<visual>
+			<origin xyz="${reflect_big_link}" rpy="0 -0.7 0" />
+       			<geometry>
+          			<box size="0.2 0.03 0.03" />
+        		</geometry>
         		<material name="red" >
-          	<color rgba="1.00 0 0 1.0"/>
+          			<color rgba="1.00 0 0 1.0"/>
        			</material>
-      </visual>
+     		</visual>
 			<inertial>
 				<mass value="10"/>
@@ -44,45 +44,45 @@
 			<collision>
 				<geometry>
-          	<box size="0.2 0.03 0.03" />
-        	</geometry>
+          				<box size="0.2 0.03 0.03" />
+        			</geometry>
 			</collision>
-		</link>
-		<joint name="body_to_${prefix}_big_leg" type="revolute">
-       <origin xyz="${reflect_big_joint}" rpy="0 0 0"/>
-        <parent link="body"/>
-        <child link="${prefix}_big_leg"/>
-				<axis xyz = "0 1 0"/>
-        <limit effort="30" velocity="1.0" lower="-2.2" upper="0.7" />
-    </joint>
+	</link>
+	<joint name="body_to_${prefix}_big_leg" type="revolute">
+       		<origin xyz="${reflect_big_joint}" rpy="0 0 0"/>
+        	<parent link="body"/>
+        	<child link="${prefix}_big_leg"/>
+		<axis xyz = "0 1 0"/>
+        	<limit effort="30" velocity="1.0" lower="-2.2" upper="0.7" />
+    	</joint>
 		<link name="${prefix}_small_leg">
 			<visual>
 				<origin xyz="${reflect_small_link}" rpy="0 0.7 0" />
-       		<geometry>
-          	<box size="0.2 0.03 0.03" />
-        	</geometry>
-        		<material name="red" >
-          	<color rgba="1.00 0 0 1.0"/>
-       			</material>
-      </visual>
-				<inertial>
-					<mass value="10"/>
-					<inertia ixx="0.4" ixy="0.0" ixz="0.0" iyy="0.4" iyz="0.0" izz="0.2"/>
-				</inertial>
+       				<geometry>
+          				<box size="0.2 0.03 0.03" />
+        			</geometry>
+        			<material name="red" >
+          				<color rgba="1.00 0 0 1.0"/>
+       				</material>
+      			</visual>
+			<inertial>
+				<mass value="10"/>
+				<inertia ixx="0.4" ixy="0.0" ixz="0.0" iyy="0.4" iyz="0.0" izz="0.2"/>
+			</inertial>
 			<collision>
 				<geometry>
-          	<box size="0.2 0.03 0.03" />
-        	</geometry>
+          				<box size="0.2 0.03 0.03" />
+        			</geometry>
 			</collision>
 		</link>
 		<joint name="${prefix}_big_leg_to_${prefix}_small_leg" type="revolute">
-       <origin xyz="${reflect_small_joint}" rpy="0 0 0"/>
-        <parent link="${prefix}_big_leg"/>
-        <child link="${prefix}_small_leg"/>
-				<axis xyz = "0 1 0"/>
-        <limit effort="30" velocity="1.0" lower="-0.7" upper="0.7" />
-    </joint>
+       			<origin xyz="${reflect_small_joint}" rpy="0 0 0"/>
+        		<parent link="${prefix}_big_leg"/>
+        		<child link="${prefix}_small_leg"/>
+			<axis xyz = "0 1 0"/>
+        		<limit effort="30" velocity="1.0" lower="-0.7" upper="0.7" />
+    		</joint>
 			<!-- A bunch of stuff cut -->
    </xacro:macro>
-		<xacro:leg prefix="left_back" reflect_big_link="-0.05 -0.05 0" reflect_big_joint="-0.15 0.2 0.2" reflect_small_link="0.05 -0.05 0" reflect_small_joint="-0.13 0.055 -0.1" />
+	<xacro:leg prefix="left_back" reflect_big_link="-0.05 -0.05 0" reflect_big_joint="-0.15 0.2 0.2" reflect_small_link="0.05 -0.05 0" reflect_small_joint="-0.13 0.055 -0.1" />
 	<xacro:leg prefix="left_forward" reflect_big_link="-0.05 -0.05 0" reflect_big_joint="0.15 0.2 0.2" reflect_small_link="0.05 -0.05 0" reflect_small_joint="-0.15 0.055 -0.1" />
 	<xacro:leg prefix="right_back" reflect_big_link="-0.05 -0.05 0" reflect_big_joint="-0.15 -0.1 0.2" reflect_small_link="0.05 -0.05 0" reflect_small_joint="-0.15 -0.055 -0.1" />

Commit message: Cool! Now update all my work with camera

File: spot/src/myrobot/urdf/thespot.urdf.xacro (robot description, xacro)
@@ -1,4 +1,5 @@
 <?xml version='1.0'?>
 	<robot name ="thespot_robot" xmlns:xacro="http://www.ros.org/wiki/xacro">
+		<xacro:include filename="$(find myrobot)/urdf/thespot.gazebo" />
 			<link name="world"/>
   			<joint name="fixed" type="fixed">
@@ -84,8 +85,8 @@
 			<!-- A bunch of stuff cut -->
    </xacro:macro>
-		<xacro:leg prefix="left_back" reflect_big_link="-0.05 -0.05 0" reflect_big_joint="-0.15 0.2 0.2" reflect_small_link="0.05 -0.05 0" reflect_small_joint="-0.13 0.055 -0.1" />
-	<xacro:leg prefix="left_forward" reflect_big_link="-0.05 -0.05 0" reflect_big_joint="0.15 0.2 0.2" reflect_small_link="0.05 -0.05 0" reflect_small_joint="-0.15 0.055 -0.1" />
-	<xacro:leg prefix="right_back" reflect_big_link="-0.05 -0.05 0" reflect_big_joint="-0.15 -0.1 0.2" reflect_small_link="0.05 -0.05 0" reflect_small_joint="-0.15 -0.055 -0.1" />
-	<xacro:leg prefix="right_forward" reflect_big_link="-0.05 -0.05 0" reflect_big_joint="0.15 -0.1 0.2" reflect_small_link="0.05 -0.05 0" reflect_small_joint="-0.15 -0.055 -0.1" />
+		<xacro:leg prefix="left_back" reflect_big_link="-0.05 -0.05 0" reflect_big_joint="-0.15 0.2 0.25" reflect_small_link="0.05 -0.05 0" reflect_small_joint="-0.13 0.055 -0.1" />
+	<xacro:leg prefix="left_forward" reflect_big_link="-0.05 -0.05 0" reflect_big_joint="0.15 0.2 0.25" reflect_small_link="0.05 -0.05 0" reflect_small_joint="-0.15 0.055 -0.1" />
+	<xacro:leg prefix="right_back" reflect_big_link="-0.05 -0.05 0" reflect_big_joint="-0.15 -0.1 0.25" reflect_small_link="0.05 -0.05 0" reflect_small_joint="-0.15 -0.055 -0.1" />
+	<xacro:leg prefix="right_forward" reflect_big_link="-0.05 -0.05 0" reflect_big_joint="0.15 -0.1 0.25" reflect_small_link="0.05 -0.05 0" reflect_small_joint="-0.15 -0.055 -0.1" />
 	<gazebo>
   		<plugin name="gazebo_ros_control" filename="libgazebo_ros_control.so">
@@ -119,3 +120,31 @@
 	<xacro:leg prefix="right_forward" reflect_big_link="-0.05 -0.05 -0.05" reflect_big_joint="-0.15 -0.1 0.2" reflect_small_link="0.05 -0.05 -0.05" reflect_small_joint="-0.15 -0.055 -0.1" />
 	<xacro:leg prefix="left_forward" reflect_big_link="-0.05 -0.05 -0.05" reflect_big_joint="0.15 -0.1 0.2" reflect_small_link="0.05 -0.05 -0.05" reflect_small_joint="-0.15 -0.055 -0.1" />
+ <!--Camera-->
+  		<link name="camera_link">
+    			<collision>
+      				<origin xyz="0 0 0" rpy="0 0.7 0"/>
+      				<geometry>
+    					<box size="0.025 0.025 0.025"/>
+     		 		</geometry>
+    			</collision>
+   			<visual>
+      				<origin xyz="0 0 0" rpy="0 0.7 0"/>
+      				<geometry>
+    					<box size="0.025 0.025 0.025"/>
+      				</geometry>
+      				<material name="0 1 0 1"/>
+    			</visual>
+    			<inertial>
+      				<mass value="1e-5" />
+      				<origin xyz="0 0 0" rpy="0 0.7 0"/>
+      				<inertia ixx="1e-6" ixy="0" ixz="0" iyy="1e-6" iyz="0" izz="1e-6" />
+    				</inertial>
+  		</link>
+		<joint name="camera_joint" type="fixed">
+    			<axis xyz="0 1 0" />
+    			<origin xyz="0.13 -0.05 -0.03" rpy="0 0 0"/>
+    			<parent link="left_back_small_leg"/>
+    			<child link="camera_link"/>
+  		</joint>
+<!--addition-->
 </robot>

Commit message: Testing work begins

File: spot/src/myrobot/urdf/thespot.urdf.xacro (robot description, xacro)
@@ -7,36 +7,36 @@
   			 	<child link="body"/>
   			</joint>
-			<link name ="body">
-				<visual>
-      					<origin xyz="0 0 0.3" rpy="0 0 0" />
-       					<geometry>
-          					<box size="0.4 0.2 0.1" />
-        				</geometry>
-        				<material name="Cyan">
-          					<color rgba="0 1.0 1.0 1.0"/>
-       					</material>
-      				</visual>
-				<inertial>
-					<mass value="5"/>
-					<inertia ixx="0.1" ixy="0.0" ixz="0.1" iyy="0.0" iyz="0.0" izz="0.1"/>
-				</inertial>
-				<collision>
-					<origin xyz="0 0 0.3" rpy="0 0 0" />
-       					<geometry>
-          					<box size="0.4 0.2 0.1" />
-        				</geometry>
-				</collision>
-			</link>
-<xacro:macro name="leg" params="prefix reflect_big_link reflect_big_joint reflect_small_link  reflect_small_joint">
-	<link name="${prefix}_big_leg">
-		<visual>
-			<origin xyz="${reflect_big_link}" rpy="0 -0.7 0" />
-       			<geometry>
-          			<box size="0.2 0.03 0.03" />
-        		</geometry>
+		<link name ="body">
+			<visual>
+      	<origin xyz="0 0 0.3" rpy="0 0 0" />
+       		<geometry>
+          	<box size="0.4 0.2 0.1" />
+        	</geometry>
+        	<material name="Cyan">
+          	<color rgba="0 1.0 1.0 1.0"/>
+       		</material>
+      </visual>
+			<inertial>
+				<mass value="5"/>
+				<inertia ixx="0.1" ixy="0.0" ixz="0.1" iyy="0.0" iyz="0.0" izz="0.1"/>
+			</inertial>
+			<collision>
+	<origin xyz="0 0 0.3" rpy="0 0 0" />
+       				<geometry>
+          	<box size="0.4 0.2 0.1" />
+        	</geometry>
+			</collision>
+		</link>
+			<xacro:macro name="leg" params="prefix reflect_big_link reflect_big_joint reflect_small_link  reflect_small_joint">
+		<link name="${prefix}_big_leg">
+			<visual>
+				<origin xyz="${reflect_big_link}" rpy="0 -0.7 0" />
+       		<geometry>
+          	<box size="0.2 0.03 0.03" />
+        	</geometry>
         		<material name="red" >
-          			<color rgba="1.00 0 0 1.0"/>
+          	<color rgba="1.00 0 0 1.0"/>
        			</material>
-     		</visual>
+      </visual>
 			<inertial>
 				<mass value="10"/>
@@ -45,53 +45,48 @@
 			<collision>
 				<geometry>
-          				<box size="0.2 0.03 0.03" />
-        			</geometry>
+          	<box size="0.2 0.03 0.03" />
+        	</geometry>
 			</collision>
-	</link>
-	<joint name="body_to_${prefix}_big_leg" type="revolute">
-       		<origin xyz="${reflect_big_joint}" rpy="0 0 0"/>
-        	<parent link="body"/>
-        	<child link="${prefix}_big_leg"/>
-		<axis xyz = "0 1 0"/>
-        	<limit effort="30" velocity="1.0" lower="-2.2" upper="0.7" />
-    	</joint>
+		</link>
+		<joint name="body_to_${prefix}_big_leg" type="revolute">
+       <origin xyz="${reflect_big_joint}" rpy="0 0 0"/>
+        <parent link="body"/>
+        <child link="${prefix}_big_leg"/>
+				<axis xyz = "0 1 0"/>
+        <limit effort="30" velocity="1.0" lower="-2.2" upper="0.7" />
+    </joint>
 		<link name="${prefix}_small_leg">
 			<visual>
 				<origin xyz="${reflect_small_link}" rpy="0 0.7 0" />
-       				<geometry>
-          				<box size="0.2 0.03 0.03" />
-        			</geometry>
-        			<material name="red" >
-          				<color rgba="1.00 0 0 1.0"/>
-       				</material>
-      			</visual>
-			<inertial>
-				<mass value="10"/>
-				<inertia ixx="0.4" ixy="0.0" ixz="0.0" iyy="0.4" iyz="0.0" izz="0.2"/>
-			</inertial>
+       		<geometry>
+          	<box size="0.2 0.03 0.03" />
+        	</geometry>
+        		<material name="red" >
+          	<color rgba="1.00 0 0 1.0"/>
+       			</material>
+      </visual>
+				<inertial>
+					<mass value="10"/>
+					<inertia ixx="0.4" ixy="0.0" ixz="0.0" iyy="0.4" iyz="0.0" izz="0.2"/>
+				</inertial>
 			<collision>
 				<geometry>
-          				<box size="0.2 0.03 0.03" />
-        			</geometry>
+          	<box size="0.2 0.03 0.03" />
+        	</geometry>
 			</collision>
 		</link>
 		<joint name="${prefix}_big_leg_to_${prefix}_small_leg" type="revolute">
-       			<origin xyz="${reflect_small_joint}" rpy="0 0 0"/>
-        		<parent link="${prefix}_big_leg"/>
-        		<child link="${prefix}_small_leg"/>
-			<axis xyz = "0 1 0"/>
-        		<limit effort="30" velocity="1.0" lower="-0.7" upper="0.7" />
-    		</joint>
+       <origin xyz="${reflect_small_joint}" rpy="0 0 0"/>
+        <parent link="${prefix}_big_leg"/>
+        <child link="${prefix}_small_leg"/>
+				<axis xyz = "0 1 0"/>
+        <limit effort="30" velocity="1.0" lower="-0.7" upper="0.7" />
+    </joint>
 			<!-- A bunch of stuff cut -->
    </xacro:macro>
-<<<< camera_adding
 		<xacro:leg prefix="left_back" reflect_big_link="-0.05 -0.05 0" reflect_big_joint="-0.15 0.2 0.25" reflect_small_link="0.05 -0.05 0" reflect_small_joint="-0.13 0.055 -0.1" />
 	<xacro:leg prefix="left_forward" reflect_big_link="-0.05 -0.05 0" reflect_big_joint="0.15 0.2 0.25" reflect_small_link="0.05 -0.05 0" reflect_small_joint="-0.15 0.055 -0.1" />
 	<xacro:leg prefix="right_back" reflect_big_link="-0.05 -0.05 0" reflect_big_joint="-0.15 -0.1 0.25" reflect_small_link="0.05 -0.05 0" reflect_small_joint="-0.15 -0.055 -0.1" />
 	<xacro:leg prefix="right_forward" reflect_big_link="-0.05 -0.05 0" reflect_big_joint="0.15 -0.1 0.25" reflect_small_link="0.05 -0.05 0" reflect_small_joint="-0.15 -0.055 -0.1" />
-	<xacro:leg prefix="left_back" reflect_big_link="-0.05 -0.05 0" reflect_big_joint="-0.15 0.2 0.2" reflect_small_link="0.05 -0.05 0" reflect_small_joint="-0.13 0.055 -0.1" />
-	<xacro:leg prefix="left_forward" reflect_big_link="-0.05 -0.05 0" reflect_big_joint="0.15 0.2 0.2" reflect_small_link="0.05 -0.05 0" reflect_small_joint="-0.15 0.055 -0.1" />
-	<xacro:leg prefix="right_back" reflect_big_link="-0.05 -0.05 0" reflect_big_joint="-0.15 -0.1 0.2" reflect_small_link="0.05 -0.05 0" reflect_small_joint="-0.15 -0.055 -0.1" />
-	<xacro:leg prefix="right_forward" reflect_big_link="-0.05 -0.05 0" reflect_big_joint="0.15 -0.1 0.2" reflect_small_link="0.05 -0.05 0" reflect_small_joint="-0.15 -0.055 -0.1" />
 	<gazebo>
   		<plugin name="gazebo_ros_control" filename="libgazebo_ros_control.so">
