Commit message: My spot can walk now

File: src/myrobot/urdf/thespot.urdf.xacro (robot description, xacro)
@@ -2,95 +2,116 @@
 	<robot name ="thespot_robot" xmlns:xacro="http://www.ros.org/wiki/xacro">
 		<xacro:include filename="$(find myrobot)/urdf/thespot.gazebo" />
-			<link name="world"/>
-  			<joint name="fixed" type="fixed">
-    				<parent link="world"/>
-  			 	<child link="body"/>
-  			</joint>
-			<link name ="body">
-				<visual>
-      					<origin xyz="0 0 0.3" rpy="0 0 0" />
-       					<geometry>
-          					<box size="0.4 0.2 0.1" />
-        				</geometry>
-        				<material name="Cyan">
-          					<color rgba="0 1.0 1.0 1.0"/>
-       					</material>
-      				</visual>
-				<inertial>
-					<mass value="5"/>
-					<inertia ixx="0.1" ixy="0.0" ixz="0.1" iyy="0.0" iyz="0.0" izz="0.1"/>
-				</inertial>
-				<collision>
-					<origin xyz="0 0 0.3" rpy="0 0 0" />
-       					<geometry>
-          					<box size="0.4 0.2 0.1" />
-        				</geometry>
-				</collision>
-			</link>
-<xacro:macro name="leg" params="prefix reflect_big_link reflect_big_joint reflect_small_link  reflect_small_joint">
-	<link name="${prefix}_big_leg">
-		<visual>
-			<origin xyz="${reflect_big_link}" rpy="0 -0.7 0" />
-       			<geometry>
-          			<box size="0.2 0.03 0.03" />
-        		</geometry>
-        		<material name="red" >
-          			<color rgba="1.00 0 0 1.0"/>
-       			</material>
-     		</visual>
+		<link name ="body">
+			<visual>
+      	<origin xyz="0 0 5.5" rpy="0 0 0" />
+       		<geometry>
+          	<box size="0.4 0.2 0.1" />
+        	</geometry>
+        	<material name="Cyan">
+          	<color rgba="0 1.0 1.0 1.0"/>
+       		</material>
+      </visual>
 			<inertial>
-				<mass value="10"/>
-				<inertia ixx="0.1" ixy="0.0" ixz="0.1" iyy="0.0" iyz="0.1" izz="0.0"/>
+				<mass value="8"/>
+					<inertia ixx="0.8" ixy="0.8" ixz="0.6" iyy="0.7" iyz="0.9" izz="0.8"/>
 			</inertial>
 			<collision>
+	<origin xyz="0 0 5.5" rpy="0 0 0" />
+       				<geometry>
+          	<box size="0.4 0.2 0.1" />
+        	</geometry>
+			</collision>
+		</link>
+		<gazebo reference="body">
+        <kp>1000.0</kp>
+        <kd>1000.0</kd>
+        <mu1>0.5</mu1>
+        <mu2>0.5</mu2>
+        <material>Gazebo/Red</material>
+    </gazebo>
+			<xacro:macro name="leg" params="prefix reflect_big_link reflect_big_joint reflect_small_link  reflect_small_joint">
+		<link name="${prefix}_big_leg">
+			<visual>
+				<origin xyz="${reflect_big_link}" rpy="0 -0.7 0" />
+       		<geometry>
+          	<box size="0.2 0.03 0.03" />
+        	</geometry>
+        		<material name="red" >
+          	<color rgba="1.00 0 0 1.0"/>
+       			</material>
+      </visual>
+			<inertial>
+				<mass value="0.2"/>
+					<inertia ixx="0.8" ixy="0.8" ixz="0.6" iyy="0.7" iyz="0.9" izz="0.8"/>
+			</inertial>
+			<collision>
+			<origin xyz="${reflect_big_link}" rpy="0 -0.7 0" />
 				<geometry>
-          				<box size="0.2 0.03 0.03" />
-        			</geometry>
+          	<box size="0.2 0.03 0.03" />
+        	</geometry>
 			</collision>
-	</link>
-	<joint name="body_to_${prefix}_big_leg" type="revolute">
-       		<origin xyz="${reflect_big_joint}" rpy="0 0 0"/>
-        	<parent link="body"/>
-        	<child link="${prefix}_big_leg"/>
-		<axis xyz = "0 1 0"/>
-        	<limit effort="30" velocity="1.0" lower="-2.2" upper="0.7" />
-    	</joint>
+		</link>
+		<gazebo reference="${prefix}_big_leg">
+        <kp>1000.0</kp>
+        <kd>1000.0</kd>
+        <mu1>50</mu1>
+        <mu2>100</mu2>
+        <material>Gazebo/Blue</material>
+    </gazebo>
+		<joint name="body_to_${prefix}_big_leg" type="revolute">
+       <origin xyz="${reflect_big_joint}" rpy="0 0 0"/>
+        <parent link="body"/>
+        <child link="${prefix}_big_leg"/>
+				<axis xyz = "0 1 0"/>
+        <limit effort="50" velocity="1.0" lower="-2.2" upper="0.7" />
+		<joint_properties damping="1.0" friction="50.0" />
+    </joint>
 		<link name="${prefix}_small_leg">
 			<visual>
 				<origin xyz="${reflect_small_link}" rpy="0 0.7 0" />
-       				<geometry>
-          				<box size="0.2 0.03 0.03" />
-        			</geometry>
-        			<material name="red" >
-          				<color rgba="1.00 0 0 1.0"/>
-       				</material>
-      			</visual>
-			<inertial>
-				<mass value="10"/>
-				<inertia ixx="0.4" ixy="0.0" ixz="0.0" iyy="0.4" iyz="0.0" izz="0.2"/>
-			</inertial>
+       		<geometry>
+          	<box size="0.25 0.03 0.03" />
+			<origin xyz="${reflect_small_link}" rpy="0 0.7 0" />
+        	</geometry>
+        		<material name="red" >
+          	<color rgba="1.00 0 0 1.0"/>
+       			</material>
+      </visual>
+				<inertial>
+					<mass value="0.2"/>
+					<inertia ixx="0.8" ixy="0.8" ixz="0.6" iyy="0.7" iyz="0.9" izz="0.8"/>
+				</inertial>
 			<collision>
+			<origin xyz="${reflect_big_joint}" rpy="0 0 0"/>
 				<geometry>
-          				<box size="0.2 0.03 0.03" />
-        			</geometry>
+          	<box size="0.25 0.03 0.03" />
+        	</geometry>
 			</collision>
 		</link>
+		<gazebo reference="${prefix}_small_leg">
+                <kp>1000.0</kp>
+        		<kd>1000.0</kd>
+        		<mu1>5000.0</mu1>
+        		<mu2>100000.0</mu2>
+                <fdir1>1 0 0</fdir1>
+                <maxContacts>1</maxContacts>
+                <minDepth>0.005</minDepth>
+                <gravity>true</gravity>
+        <material>Gazebo/Black</material>
+        </gazebo>
 		<joint name="${prefix}_big_leg_to_${prefix}_small_leg" type="revolute">
-       			<origin xyz="${reflect_small_joint}" rpy="0 0 0"/>
-        		<parent link="${prefix}_big_leg"/>
-        		<child link="${prefix}_small_leg"/>
-			<axis xyz = "0 1 0"/>
-        		<limit effort="30" velocity="1.0" lower="-0.7" upper="0.7" />
-    		</joint>
+       <origin xyz="${reflect_small_joint}" rpy="0 0 0"/>
+        <parent link="${prefix}_big_leg"/>
+        <child link="${prefix}_small_leg"/>
+				<axis xyz = "0 1 0"/>
+        <limit effort="30" velocity="1.0" lower="-0.7" upper="0.7" />
+		<joint_properties damping="1.0" friction="50.0" />
+    </joint>
 			<!-- A bunch of stuff cut -->
-   </xacro:macro>
-		<xacro:leg prefix="left_back" reflect_big_link="-0.05 -0.05 0" reflect_big_joint="-0.15 0.2 0.25" reflect_small_link="0.05 -0.05 0" reflect_small_joint="-0.13 0.055 -0.1" />
-	<xacro:leg prefix="left_forward" reflect_big_link="-0.05 -0.05 0" reflect_big_joint="0.15 0.2 0.25" reflect_small_link="0.05 -0.05 0" reflect_small_joint="-0.15 0.055 -0.1" />
-	<xacro:leg prefix="right_back" reflect_big_link="-0.05 -0.05 0" reflect_big_joint="-0.15 -0.1 0.25" reflect_small_link="0.05 -0.05 0" reflect_small_joint="-0.15 -0.055 -0.1" />
-	<xacro:leg prefix="right_forward" reflect_big_link="-0.05 -0.05 0" reflect_big_joint="0.15 -0.1 0.25" reflect_small_link="0.05 -0.05 0" reflect_small_joint="-0.15 -0.055 -0.1" />
-	<xacro:leg prefix="left_back" reflect_big_link="-0.05 -0.05 0" reflect_big_joint="-0.15 0.2 0.2" reflect_small_link="0.05 -0.05 0" reflect_small_joint="-0.13 0.055 -0.1" />
-	<xacro:leg prefix="left_forward" reflect_big_link="-0.05 -0.05 0" reflect_big_joint="0.15 0.2 0.2" reflect_small_link="0.05 -0.05 0" reflect_small_joint="-0.15 0.055 -0.1" />
-	<xacro:leg prefix="right_back" reflect_big_link="-0.05 -0.05 0" reflect_big_joint="-0.15 -0.1 0.2" reflect_small_link="0.05 -0.05 0" reflect_small_joint="-0.15 -0.055 -0.1" />
-	<xacro:leg prefix="right_forward" reflect_big_link="-0.05 -0.05 0" reflect_big_joint="0.15 -0.1 0.2" reflect_small_link="0.05 -0.05 0" reflect_small_joint="-0.15 -0.055 -0.1" />
+    </xacro:macro>
+		<xacro:leg prefix="left_back" reflect_big_link="-0.05 -0.05 0" reflect_big_joint="-0.15 0.2 5.45" reflect_small_link="0.05 -0.05 0" reflect_small_joint="-0.13 0.055 -0.1" />
+	<xacro:leg prefix="left_forward" reflect_big_link="-0.05 -0.05 0" reflect_big_joint="0.15 0.2 5.45" reflect_small_link="0.05 -0.05 0" reflect_small_joint="-0.15 0.055 -0.1" />
+	<xacro:leg prefix="right_back" reflect_big_link="-0.05 -0.05 0" reflect_big_joint="-0.15 -0.1 5.45" reflect_small_link="0.05 -0.05 0" reflect_small_joint="-0.15 -0.055 -0.1" />
+	<xacro:leg prefix="right_forward" reflect_big_link="-0.05 -0.05 0" reflect_big_joint="0.15 -0.1 5.45" reflect_small_link="0.05 -0.05 0" reflect_small_joint="-0.15 -0.055 -0.1" />
 	<gazebo>
   		<plugin name="gazebo_ros_control" filename="libgazebo_ros_control.so">
@@ -119,10 +140,10 @@
     		</actuator>
   		</transmission>
-	</xacro:macro>
-		<xacro:leg prefix="left_back" reflect_big_link="-0.05 -0.05 -0.05" reflect_big_joint="-0.15 0.2 0.2" reflect_small_link="0.05 -0.05 -0.05" reflect_small_joint="-0.13 0.055 -0.1" />
-	<xacro:leg prefix="right_back" reflect_big_link="-0.05 -0.05 -0.05" reflect_big_joint="0.15 0.2 0.2" reflect_small_link="0.05 -0.05 -0.05" reflect_small_joint="-0.15 0.055 -0.1" />
-	<xacro:leg prefix="right_forward" reflect_big_link="-0.05 -0.05 -0.05" reflect_big_joint="-0.15 -0.1 0.2" reflect_small_link="0.05 -0.05 -0.05" reflect_small_joint="-0.15 -0.055 -0.1" />
-	<xacro:leg prefix="left_forward" reflect_big_link="-0.05 -0.05 -0.05" reflect_big_joint="0.15 -0.1 0.2" reflect_small_link="0.05 -0.05 -0.05" reflect_small_joint="-0.15 -0.055 -0.1" />
- <!--Camera-->
+	 </xacro:macro>
+		<xacro:leg prefix="left_back" reflect_big_link="-0.05 -0.05 1" reflect_big_joint="-0.15 0.2 10.45" reflect_small_link="0.05 -0.05 0.15" reflect_small_joint="-0.13 0.055 2" />
+	<xacro:leg prefix="left_forward" reflect_big_link="-0.05 -0.05 1" reflect_big_joint="0.15 0.2 10.45" reflect_small_link="0.05 -0.05 0.15" reflect_small_joint="-0.15 0.055 2" />
+	<xacro:leg prefix="right_back" reflect_big_link="-0.05 -0.05 1" reflect_big_joint="-0.15 -0.1 10.45" reflect_small_link="0.05 -0.05 0.15" reflect_small_joint="-0.15 -0.055 2" />
+	<xacro:leg prefix="right_forward" reflect_big_link="-0.05 -0.05 1" reflect_big_joint="0.15 -0.1 10.45" reflect_small_link="0.05 -0.05 0.15" reflect_small_joint="-0.15 -0.055 2" />
+	<!--Camera-->
   		<link name="camera_link">
     			<collision>
@@ -151,4 +172,82 @@
     			<child link="camera_link"/>
   		</joint>
+		  <link name="camera_link1">
+    			<collision>
+      				<origin xyz="0 0 0" rpy="0 0.7 0"/>
+      				<geometry>
+    					<box size="0.025 0.025 0.025"/>
+     		 		</geometry>
+    			</collision>
+   			<visual>
+      				<origin xyz="0 0 0" rpy="0 0.7 0"/>
+      				<geometry>
+    					<box size="0.025 0.025 0.025"/>
+      				</geometry>
+      				<material name="0 1 0 1"/>
+    			</visual>
+    			<inertial>
+      				<mass value="1e-5" />
+      				<origin xyz="0 0 0" rpy="0 0.7 0"/>
+      				<inertia ixx="1e-6" ixy="0" ixz="0" iyy="1e-6" iyz="0" izz="1e-6" />
+    				</inertial>
+  		</link>
+		<joint name="camera_joint1" type="fixed">
+    			<axis xyz="0 1 0" />
+    			<origin xyz="0.13 -0.05 -0.03" rpy="0 0 0"/>
+    			<parent link="left_forward_small_leg"/>
+    			<child link="camera_link1"/>
+  		</joint>
+		  <link name="camera_link2">
+    			<collision>
+      				<origin xyz="0 0 0" rpy="0 0.7 0"/>
+      				<geometry>
+    					<box size="0.025 0.025 0.025"/>
+     		 		</geometry>
+    			</collision>
+   			<visual>
+      				<origin xyz="0 0 0" rpy="0 0.7 0"/>
+      				<geometry>
+    					<box size="0.025 0.025 0.025"/>
+      				</geometry>
+      				<material name="0 1 0 1"/>
+    			</visual>
+    			<inertial>
+      				<mass value="1e-5" />
+      				<origin xyz="0 0 0" rpy="0 0.7 0"/>
+      				<inertia ixx="1e-6" ixy="0" ixz="0" iyy="1e-6" iyz="0" izz="1e-6" />
+    				</inertial>
+  		</link>
+		<joint name="camera_joint2" type="fixed">
+    			<axis xyz="0 1 0" />
+    			<origin xyz="0.13 -0.05 -0.03" rpy="0 0 0"/>
+    			<parent link="right_back_small_leg"/>
+    			<child link="camera_link2"/>
+  		</joint>
+		  <link name="camera_link3">
+    			<collision>
+      				<origin xyz="0 0 0" rpy="0 0.7 0"/>
+      				<geometry>
+    					<box size="0.025 0.025 0.025"/>
+     		 		</geometry>
+    			</collision>
+   			<visual>
+      				<origin xyz="0 0 0" rpy="0 0.7 0"/>
+      				<geometry>
+    					<box size="0.025 0.025 0.025"/>
+      				</geometry>
+      				<material name="0 1 0 1"/>
+    			</visual>
+    			<inertial>
+      				<mass value="1e-5" />
+      				<origin xyz="0 0 0" rpy="0 0.7 0"/>
+      				<inertia ixx="1e-6" ixy="0" ixz="0" iyy="1e-6" iyz="0" izz="1e-6" />
+    				</inertial>
+  		</link>
+		<joint name="camera_joint3" type="fixed">
+    			<axis xyz="0 1 0" />
+    			<origin xyz="0.13 -0.05 -0.03" rpy="0 0 0"/>
+    			<parent link="right_forward_small_leg"/>
+    			<child link="camera_link3"/>
+  		</joint>
 <!--addition-->
 </robot>
